File: bmp_x6.kicad_pcb (KiCad board)
At the start: 2 copper layers, 50 x 50 mm, 67 parts, among them J1 USB_B, J2 Conn_01x05_Pin, J3 Conn_02x05_Odd_Even, Q1 NMOS, Q2 PMOS, Q3 PMOS, Q4 NMOS, SW1 SW_Push, U1 STM32F103CBTx, U2 USB6B1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

Commit message: components relocated.
Parts:
- moved C1 47.0 mm to (70.3, 58.9)
- moved R1 47.0 mm to (72.1, 58.9)
- moved R22 25.3 mm to (30.2, 47.9), turned to 180 degrees
- moved R19 16.8 mm to (34.9, 43.6), turned to -90 degrees
- moved R18 16.1 mm to (29.5, 43.6), turned to 90 degrees
- moved R20 15.8 mm to (41.5, 44.3)
- moved R23 15.0 mm to (37.0, 47.2), turned to 90 degrees
- moved Q2 14.1 mm to (32.2, 43.0)
- moved Q3 13.7 mm to (37.8, 43.4), turned to 0 degrees
- moved C20 13.3 mm to (45.8, 55.4)
- moved C8 13.1 mm to (30.6, 29.4), turned to 180 degrees
- moved U5 12.5 mm to (43.5, 56.2), turned to -90 degrees
- moved C7 12.4 mm to (33.9, 27.2), turned to 0 degrees
- moved C21 12.0 mm to (41.0, 55.4)
- moved R12 11.4 mm to (70.1, 67.2)
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Connections:
- J3 pad 6: GND -> /io/xTXD
- J3 pad 9: /io/xVCC -> xVCC
- Q2 pad 1: /io/xVCC -> xVCC
- R18 pad 2: /io/xVCC -> xVCC
- R9 pad 2: TPWR -> xVCC
- U4 pad 6: GND -> /io/xTXD
Routing:
- net +3.3V: track 18.6 -> 0.00 mm
- net Net-(U1-PD0): track 13.6 -> 0.00 mm
- net /mcu/USBX2_DM: track 12.3 -> 0.00 mm
- net /mcu/USBX2_DP: track 12.1 -> 0.00 mm
- net /mcu/USBX1_DP: track 11.6 -> 0.00 mm, vias 2 -> 0
- net /mcu/USBX1_DM: track 11.1 -> 0.00 mm, vias 2 -> 0
- net Net-(U1-PD1): track 10.3 -> 0.35 mm
- net /mcu/VER_2: track 8.22 -> 0.00 mm, vias 1 -> 0
- net /mcu/VER_1: track 7.58 -> 0.00 mm, vias 1 -> 0
- net /mcu/VER_0: track 7.08 -> 0.03 mm, vias 1 -> 0
- net /mcu/OWN_SWDIO: track 3.84 -> 0.00 mm
- net /mcu/OWN_SWCLK: track 3.31 -> 0.00 mm

Commit message: drawing continue...
Parts:
- moved R18 7.47 mm to (28.6, 51.0), turned to -90 degrees
- moved R22 3.82 mm to (33.7, 49.6), turned to 0 degrees
- moved C10 1.91 mm to (70.9, 50.9)
- moved C12 1.91 mm to (70.9, 49.1)
- moved C13 1.31 mm to (65.9, 63.7)
- moved C9 1.13 mm to (66.1, 61.8)
- moved C11 1.07 mm to (57.6, 48.5)
- moved C14 0.49 mm to (55.3, 50.7)
- moved U2 0.16 mm to (57.2, 40.9)
Routing:
- net /mcu/iBTN: track 0.00 -> 76.6 mm, vias 0 -> 1
- net xTPWR: track 0.00 -> 37.4 mm, vias 0 -> 4
- net +5V: track 0.00 -> 33.5 mm
- net +3.3V: track 0.00 -> 33.4 mm
- net Net-(J1-GND): track 0.00 -> 24.1 mm
- net xVCC: track 0.03 -> 23.4 mm, vias 0 -> 2
- net /mcu/USBX2_DP: track 0.00 -> 13.2 mm
- net /mcu/USBX1_DP: track 0.00 -> 12.6 mm, vias 0 -> 2
- net /mcu/USBX2_DM: track 0.00 -> 12.2 mm
- net Net-(J1-VBUS): track 0.00 -> 11.9 mm
- net /mcu/USBX1_DM: track 0.00 -> 11.8 mm, vias 0 -> 2
- net Net-(R6-Pad2): track 0.00 -> 10.2 mm
- net Net-(R5-Pad2): track 0.00 -> 8.40 mm
- net Net-(Q2-G): track 0.00 -> 8.19 mm
- net Net-(Q2-S): track 0.00 -> 7.46 mm
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
Commit message: drawing continue..
Parts:
- moved R12 31.8 mm to (50.2, 42.4), turned to -90 degrees
- moved R14 30.6 mm to (48.7, 42.4), turned to -90 degrees
- moved R13 29.8 mm to (51.8, 42.4), turned to -90 degrees
- moved C11 8.57 mm to (54.6, 56.5)
- moved C12 2.18 mm to (69.0, 50.2)
- moved C10 2.11 mm to (69.0, 51.8)
- moved R18 1.60 mm to (28.6, 49.4)
- moved R11 1.52 mm to (60.7, 63.3), turned to 90 degrees
- turned U4 to -90 degrees
Connections:
- U4 pad 3: iTXD -> iTxD
- U6 pad 3: iRXD -> iRxD
Routing:
- net +3.3V: track 33.4 -> 168.6 mm, vias 0 -> 8
- net /mcu/LED0: track 0.00 -> 90.7 mm, vias 0 -> 2
- net /mcu/LED1: track 0.00 -> 88.4 mm, vias 0 -> 2
- net /mcu/LED2: track 0.00 -> 81.9 mm, vias 0 -> 2
- net iRST_SENSE: track 4.58 -> 46.0 mm, vias 0 -> 2
- net /io/xRST: track 6.43 -> 40.6 mm, vias 0 -> 1
- net xVCC: track 23.4 -> 50.7 mm, vias 2 -> 4
- net /mcu/T_PWR_SENSE: track 0.00 -> 25.8 mm
- net /io/xRXD: track 0.00 -> 22.2 mm
- net iRxD: track 0.00 -> 20.1 mm
- net /mcu/USBX1_H: track 0.00 -> 18.4 mm, vias 0 -> 2
- net /mcu/OWN_SWDIO: track 0.00 -> 18.4 mm
- net /mcu/VER_2: track 0.00 -> 16.3 mm
- net iTDO: track 0.00 -> 16.2 mm
- net /io/xTDI: track 0.00 -> 16.2 mm, vias 0 -> 1
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