File: bmp_x6.kicad_pcb (KiCad board)
At the start: 2 copper layers, 50 x 50 mm, 67 parts, among them J1 USB_B, J2 Conn_01x05_Pin, J3 Conn_02x05_Odd_Even, Q1 NMOS, Q2 PMOS, Q3 PMOS, Q4 NMOS, SW1 SW_Push, U1 STM32F103CBTx, U2 USB6B1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

Commit message: update
Parts:
- removed U2: USB6B1, Package_SO:SOIC-8_3.9x4.9mm_P1.27mm
- added U8: NUP2202, Package_TO_SOT_SMD:SOT-363_SC-70-6, F.Cu at (57.4, 41.1)
Connections:
- R5 pad 2: Net-(R5-Pad2) -> /mcu/USBX2_DP
- R6 pad 2: Net-(R6-Pad2) -> /mcu/USBX2_DM
- R8 pad 2: Net-(R5-Pad2) -> /mcu/USBX2_DP
Routing:
- net Net-(R5-Pad2): track 14.1 -> 0.00 mm
- net /mcu/USBX2_DP: track 13.1 -> 26.5 mm
- net Net-(R6-Pad2): track 12.7 -> 0.00 mm
- net /mcu/USBX2_DM: track 12.1 -> 24.6 mm
- net +5V: track 40.1 -> 38.0 mm, vias 0 -> 2
Other:
- board text added: "BMP V2_1E REV-A ENIS ASLAN 2025"
- board text removed: "071224 XE6 R0"
- board text removed: "BMP V2_1E"

Commit message: order data git add .!
Other:
- board text removed: "ENIS ASLAN"
Changed lines of the file:
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@@
 			(outputformat 1)
 			(mirror no)
-			(drillshape 1)
+			(drillshape 0)
 			(scaleselection 1)
-			(outputdirectory "")
+			(outputdirectory "/home/enis/Desktop/bmp/bmp_x6/output/")
 		)
 	)
@@
 				)
 			)
-		)
-	)
-	(gr_text "ENIS ASLAN"
-		(at 64.3406 68.7212 0)
-		(layer "F.SilkS")
-		(effects
-			(font
-				(face "Arial")
-				(size 0.8 0.8)
-				(thickness 0.2)
-				(bold yes)
-			)
-			(justify left bottom)
-		)
-		(render_cache "ENIS ASLAN" 0
-			(polygon
-				(pts
-					(xy 64.415484 68.5852) (xy 64.415484 67.816128) (xy 65.020962 67.816128) (xy 65.020962 67.94074)
-					(xy 64.576685 67.94074) (xy 64.576685 68.135011) (xy 64.987648 68.135011) (xy 64.987648 68.259624)
-					(xy 64.576685 68.259624) (xy 64.576685 68.460587) (xy 65.043384 68.460587) (xy 65.043384 68.5852)
-				)
-			)
-			(polygon
-				(pts
-					(xy 65.630788 68.5852) (xy 65.295198 67.992959) (xy 65.302898 68.075054) (xy 65.305066 68.131592)
-					(xy 65.305066 68.5852) (xy 65.16189 68.5852) (xy 65.16189 67.816128) (xy 65.34605 67.816128) (xy 65.686524 68.413253)
-					(xy 65.678993 68.332506) (xy 65.676657 68.263141) (xy 65.676657 67.816128) (xy 65.819832 67.816128)
-					(xy 65.819832 68.5852)
-				)
-			)
-			(polygon
-				(pts
-					(xy 65.970041 68.5852) (xy 65.970041 67.816128) (xy 66.131242 67.816128) (xy 66.131242 68.5852)
-				)
-			)
-			(polygon
-				(pts
-					(xy 66.909008 68.364404) (xy 66.903407 68.419422) (xy 66.887492 68.465531) (xy 66.861668 68.504594)
-					(xy 66.825087 68.537768) (xy 66.782519 68.562095) (xy 66.728936 68.580866) (xy 66.66199 68.593204)
-					(xy 66.578939 68.597705) (xy 66.50337 68.593846) (xy 66.440751 68.583146) (xy 66.389093 68.566676)
-					(xy 66.346664 68.545144) (xy 66.308649 68.515773) (xy 66.278217 68.480044) (xy 66.254803 68.437164)
-					(xy 66.238464 68.385848) (xy 66.394242 68.360105) (xy 66.408739 68.39848) (xy 66.429279 68.427643)
-					(xy 66.455987 68.449254) (xy 66.487858 68.463763) (xy 66.529468 68.473388) (xy 66.583286 68.476951)
-					(xy 66.643726 68.472876) (xy 66.686702 68.462248) (xy 66.716449 68.446834) (xy 66.736232 68.427393)
-					(xy 66.748017 68.403521) (xy 66.752156 68.373734) (xy 66.747143 68.343286) (xy 66.732763 68.319512)
-					(xy 66.710367 68.300583) (xy 66.678101 68.28395) (xy 66.634515 68.27023) (xy 66.54284 68.249414)
-					(xy 66.422574 68.216832) (xy 66.389898 68.20321) (xy 66.361367 68.187816) (xy 66.33595 68.16927)
-					(xy 66.314912 68.147565) (xy 66.298107 68.122305) (xy 66.285163 68.092269) (xy 66.277316 68.059088)
-					(xy 66.274514 68.019387) (xy 66.279728 67.968704) (xy 66.294562 67.926143) (xy 66.318679 67.889995)
-					(xy 66.352916 67.859212) (xy 66.392726 67.836603) (xy 66.442566 67.819195) (xy 66.504535 67.807779)
-					(xy 66.581088 67.803622) (xy 66.655049 67.807095) (xy 66.713878 67.816534) (xy 66.760164 67.83071)
-					(xy 66.796168 67.848758) (xy 66.827926 67.874023) (xy 66.853884 67.90644) (xy 66.874294 67.947165)
-					(xy 66.888785 67.997893) (xy 66.732519 68.019338) (xy 66.721334 67.987637) (xy 66.705046 67.962707)
-					(xy 66.683572 67.943378) (xy 66.657682 67.930011) (xy 66.623233 67.921134) (xy 66.577864 67.91783)
-					(xy 66.517216 67.922904) (xy 66.477004 67.935846) (xy 66.451399 67.954479) (xy 66.436566 67.978613)
-					(xy 66.431367 68.010105) (xy 66.435465 68.038126) (xy 66.44695 68.059393) (xy 66.465386 68.076475)
-					(xy 66.493112 68.091975) (xy 66.531802 68.104992) (xy 66.617187 68.125632) (xy 66.719869 68.150419)
-					(xy 66.775945 68.169205) (xy 66.820231 68.191737) (xy 66.851611 68.215758) (xy 66.876131 68.244765)
-					(xy 66.894256 68.279261) (xy 66.905141 68.318016)
-				)
-			)
-			(polygon
-				(pts
-					(xy 68.000237 68.5852) (xy 67.840648 68.5852) (xy 67.772358 68.387656) (xy 67.478876 68.387656)
-					(xy 67.410586 68.5852) (xy 67.249385 68.5852) (xy 67.365848 68.266316) (xy 67.514975 68.266316)
-					(xy 67.736308 68.266316) (xy 67.660348 68.045862) (xy 67.636852 67.971808) (xy 67.625373 67.934243)
-					(xy 67.6221 67.946211) (xy 67.60896 67.990859) (xy 67.514975 68.266316) (xy 67.365848 68.266316)
-					(xy 67.530265 67.816128) (xy 67.720432 67.816128)
-				)
-			)
-			(polygon
-				(pts
-					(xy 68.732428 68.364404) (xy 68.726827 68.419422) (xy 68.710912 68.465531) (xy 68.685087 68.504594)
-					(xy 68.648506 68.537768) (xy 68.605939 68.562095) (xy 68.552355 68.580866) (xy 68.485409 68.593204)
-					(xy 68.402358 68.597705) (xy 68.326789 68.593846) (xy 68.26417 68.583146) (xy 68.212512 68.566676)
-					(xy 68.170083 68.545144) (xy 68.132069 68.515773) (xy 68.101636 68.480044) (xy 68.078222 68.437164)
-					(xy 68.061884 68.385848) (xy 68.217662 68.360105) (xy 68.232159 68.39848) (xy 68.252699 68.427643)
-					(xy 68.279406 68.449254) (xy 68.311278 68.463763) (xy 68.352887 68.473388) (xy 68.406706 68.476951)
-					(xy 68.467145 68.472876) (xy 68.510121 68.462248) (xy 68.539868 68.446834) (xy 68.559651 68.427393)
-					(xy 68.571437 68.403521) (xy 68.575575 68.373734) (xy 68.570562 68.343286) (xy 68.556182 68.319512)
-					(xy 68.533787 68.300583) (xy 68.501521 68.28395) (xy 68.457934 68.27023) (xy 68.366259 68.249414)
-					(xy 68.245994 68.216832) (xy 68.213317 68.20321) (xy 68.184787 68.187816) (xy 68.15937 68.16927)
-					(xy 68.138332 68.147565) (xy 68.121526 68.122305) (xy 68.108583 68.092269) (xy 68.100735 68.059088)
-					(xy 68.097934 68.019387) (xy 68.103148 67.968704) (xy 68.117982 67.926143) (xy 68.142099 67.889995)
-					(xy 68.176336 67.859212) (xy 68.216146 67.836603) (xy 68.265985 67.819195) (xy 68.327954 67.807779)
-					(xy 68.404507 67.803622) (xy 68.478468 67.807095) (xy 68.537298 67.816534) (xy 68.583584 67.83071)
-					(xy 68.619588 67.848758) (xy 68.651345 67.874023) (xy 68.677304 67.90644) (xy 68.697713 67.947165)
-					(xy 68.712205 67.997893) (xy 68.555938 68.019338) (xy 68.544753 67.987637) (xy 68.528466 67.962707)
-					(xy 68.506992 67.943378) (xy 68.481101 67.930011) (xy 68.446652 67.921134) (xy 68.401283 67.91783)
-					(xy 68.340635 67.922904) (xy 68.300423 67.935846) (xy 68.274819 67.954479) (xy 68.259986 67.978613)
-					(xy 68.254787 68.010105) (xy 68.258884 68.038126) (xy 68.270369 68.059393) (xy 68.288805 68.076475)
-					(xy 68.316531 68.091975) (xy 68.355222 68.104992) (xy 68.440606 68.125632) (xy 68.543288 68.150419)
-					(xy 68.599364 68.169205) (xy 68.64365 68.191737) (xy 68.675031 68.215758) (xy 68.699551 68.244765)
-					(xy 68.717676 68.279261) (xy 68.728561 68.318016)
-				)
-			)
-			(polygon
-				(pts
-					(xy 68.850934 68.5852) (xy 68.850934 67.816128) (xy 69.012135 67.816128) (xy 69.012135 68.460587)
-					(xy 69.425296 68.460587) (xy 69.425296 68.5852)
-				)
-			)
-			(polygon
-				(pts
-					(xy 70.238673 68.5852) (xy 70.079085 68.5852) (xy 70.010795 68.387656) (xy 69.717313 68.387656)
-					(xy 69.649022 68.5852) (xy 69.487822 68.5852) (xy 69.604284 68.266316) (xy 69.753412 68.266316)
-					(xy 69.974745 68.266316) (xy 69.898785 68.045862) (xy 69.875289 67.971808) (xy 69.86381 67.934243)
-					(xy 69.860537 67.946211) (xy 69.847396 67.990859) (xy 69.753412 68.266316) (xy 69.604284 68.266316)
-					(xy 69.768701 67.816128) (xy 69.958869 67.816128)
-				)
-			)
-			(polygon
-				(pts
-					(xy 70.811863 68.5852) (xy 70.476273 67.992959) (xy 70.483972 68.075054) (xy 70.48614 68.131592)
-					(xy 70.48614 68.5852) (xy 70.342965 68.5852) (xy 70.342965 67.816128) (xy 70.527124 67.816128)
-					(xy 70.867599 68.413253) (xy 70.860067 68.332506) (xy 70.857731 68.263141) (xy 70.857731 67.816128)
-					(xy 71.000907 67.816128) (xy 71.000907 68.5852)
-				)
-			)
